File: pyIMU-GPS/pyIMU_GPS.sch (EAGLE design)
At the start: 37 parts, among them J1 TSW-108-02-S-S-MOD, J2 TSW-108-02-S-S-MOD, J3 22-27-2031-03, J4 BU-SMA-V, J5 TSW-102-02-S-S, U1 BMP180, U2 MPU-9150, U3 FGPMMOPA6H, U5 MAX4173, U6 MCP1802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

Commit message: Add mounting hole to board, move MPU_INT from XY8 to XY5, enlarge board slightly, shift GPS module and some other small changes
Parts:
- added J6: (no value), pyIMU_GPS:TSW-104-02-S-S
Connections:
- removed net XY-5: J2-5.1
- removed net XY-8/MPU_INT: J2-8.1, U2.INT
- new net XY-5/MPU_INT: J2-5.1, U2.INT
- new net XY-8: J2-8.1, J6-1.1
- net 3V3: now also C11.1; no longer C9.1
- net GND: now also J6-4.1
- net VBACK: now also C9.1; no longer C11.1
- net XY-6: now also J6-3.1
- net XY-7: now also J6-2.1
Other:
- note added: "3.3V LDO output connects directly to C11 on board. If layout is rearranged, LDO output should get its own 100nF bypass capacitor."
- note added: "FGPMMOPA6H integrated GPS receiver module from GlobalTop, based on MediaTek MT3339 GPS chipset. RTCM is a serial input for external Differential GPS data, not enabled in default firmware. Note that DGPS capability is provided by SBAS signal (WAAS, EGNOS, GAGAN, MSAS) which requires no external input."
- note removed: "3.3V LDO output connects directly to C9 on board. If layout is rearranged, LDO output should get its own 100nF bypass capacitor."
- note removed: "FGPMMOPA6H integrated GPS receiver module from GlobalTop, based on MediaTek MT3339 GPS chipset. RTCM is a serial input for external Differential GPS data, not enabled in default firmware. Note that DGPS capability is provided by SBAS signal (WAAS, EGNO, GAGAN, MSAS) which requires no external input."
- moved on the sheet: C11, C9
Changed lines of the file:
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@@
 <part name="GND6" library="supply1" deviceset="GND" device=""/>
 <part name="R4" library="rcl" deviceset="R-US_" device="R0603" value="4.7K"/>
-<part name="C9" library="rcl" deviceset="C-EU" device="C0603K" value="0.1uF"/>
+<part name="C11" library="rcl" deviceset="C-EU" device="C0603K" value="0.1uF"/>
 <part name="J3" library="pyIMU_GPS" deviceset="22-?-03" device="27-2031"/>
 <part name="U5" library="custom" deviceset="MAX4173" device="" value="MAX4173"/>
@@
 <part name="B1" library="custom" deviceset="BATT_HOLDER" device="K3000"/>
 <part name="GND16" library="supply1" deviceset="GND" device=""/>
-<part name="C11" library="rcl" deviceset="C-EU" device="C0603K" value="0.1uF"/>
+<part name="C9" library="rcl" deviceset="C-EU" device="C0603K" value="0.1uF"/>
 <part name="C13" library="rcl" deviceset="C-EU" device="C0603K" value="0.1uF"/>
 <part name="C14" library="rcl" deviceset="C-EU" device="C0603K" value="0.1uF"/>
@@
 <part name="C15" library="rcl" deviceset="C-EU" device="C0603K" value="0.1uF"/>
 <part name="GND21" library="supply1" deviceset="GND" device=""/>
+<part name="J6" library="pyIMU_GPS" deviceset="TSW-104-02-S-S" device=""/>
 </parts>
 <sheets>
@@
 data, not enabled in default firmware.
 Note that DGPS capability is provided by SBAS signal
-(WAAS, EGNO, GAGAN, MSAS) which requires no external input.</text>
+(WAAS, EGNOS, GAGAN, MSAS) which requires no external input.</text>
 <text x="114.3" y="43.18" size="2.1844" layer="97">When VBAT=11.2V,
 voltage to ADC ~ VBAT/6 = 1.87V</text>
@@
 B- connects to battery negative terminal.</text>
 <text x="12.7" y="137.16" size="2.1844" layer="97">3.3V LDO output connects directly
-to C9 on board. If layout is rearranged,
+to C11 on board. If layout is rearranged,
 LDO output should get its own 100nF
 bypass capacitor.</text>
@@
 <attribute name="VALUE" x="179.07" y="82.804" size="1.778" layer="96"/>
 </instance>
-<instance part="C9" gate="G$1" x="154.94" y="83.82"/>
+<instance part="C11" gate="G$1" x="154.94" y="83.82"/>
 <instance part="J3" gate="-1" x="73.66" y="33.02" smashed="yes" rot="MR0">
 <attribute name="NAME" x="73.66" y="29.718" size="1.524" layer="95" rot="MR0"/>
@@
 <instance part="B1" gate="G$1" x="162.56" y="124.46" rot="R90"/>
 <instance part="GND16" gate="1" x="162.56" y="116.84"/>
-<instance part="C11" gate="G$1" x="170.18" y="129.54"/>
+<instance part="C9" gate="G$1" x="170.18" y="129.54"/>
 <instance part="C13" gate="G$1" x="101.6" y="38.1" rot="R90"/>
 <instance part="C14" gate="G$1" x="63.5" y="20.32"/>
@@
 <instance part="C15" gate="G$1" x="81.28" y="55.88"/>
 <instance part="GND21" gate="1" x="81.28" y="45.72"/>
+<instance part="J6" gate="-1" x="63.5" y="175.26"/>
+<instance part="J6" gate="-2" x="63.5" y="172.72"/>
+<instance part="J6" gate="-3" x="63.5" y="170.18"/>
+<instance part="J6" gate="-4" x="63.5" y="167.64"/>
 </instances>
 <busses>
@@
 <wire x1="170.18" y1="81.28" x2="170.18" y2="86.36" width="0.1524" layer="91"/>
 <junction x="170.18" y="86.36"/>
-<pinref part="C9" gate="G$1" pin="1"/>
+<pinref part="C11" gate="G$1" pin="1"/>
 <junction x="154.94" y="86.36"/>
 </segment>
@@
 <wire x1="154.94" y1="63.5" x2="154.94" y2="78.74" width="0.1524" layer="91"/>
 <junction x="154.94" y="63.5"/>
-<pinref part="C9" gate="G$1" pin="2"/>
+<pinref part="C11" gate="G$1" pin="2"/>
 </segment>
 <segment>
@@
 <pinref part="GND16" gate="1" pin="GND"/>
 <junction x="162.56" y="119.38"/>
-<pinref part="C11" gate="G$1" pin="2"/>
+<pinref part="C9" gate="G$1" pin="2"/>
 <wire x1="170.18" y1="119.38" x2="162.56" y2="119.38" width="0.1524" layer="91"/>
 <wire x1="170.18" y1="124.46" x2="170.18" y2="119.38" width="0.1524" layer="91"/>
@@
 <wire x1="81.28" y1="48.26" x2="81.28" y2="50.8" width="0.1524" layer="91"/>
 </segment>
-</net>
-<net name="XY-8/MPU_INT" class="0">
-<segment>
-<pinref part="U2" gate="G$1" pin="INT"/>
-<wire x1="144.78" y1="190.5" x2="149.86" y2="190.5" width="0.1524" layer="91"/>
-<label x="149.86" y="190.5" size="1.778" layer="95" xref="yes"/>
-</segment>
+<segment>
+<wire x1="60.96" y1="167.64" x2="55.88" y2="167.64" width="0.1524" layer="91"/>
+<pinref part="J6" gate="-4" pin="1"/>
+<label x="55.88" y="167.64" size="1.27" layer="95" rot="R180" xref="yes"/>
+</segment>
+</net>
+<net name="XY-8" class="0">
 <segment>
 <wire x1="55.88" y1="182.88" x2="60.96" y2="182.88" width="0.1524" layer="91"/>
 <pinref part="J2" gate="-8" pin="1"/>
 <label x="55.88" y="182.88" size="1.27" layer="95" rot="R180" xref="yes"/>
+</segment>
+<segment>
+<wire x1="55.88" y1="175.26" x2="60.96" y2="175.26" width="0.1524" layer="91"/>
+<pinref part="J6" gate="-1" pin="1"/>
+<label x="55.88" y="175.26" size="1.27" layer="95" rot="R180" xref="yes"/>
 </segment>
 </net>
@@
 </segment>
 </net>
-<net name="XY-5" class="0">
+<net name="XY-5/MPU_INT" class="0">
 <segment>
 <pinref part="J2" gate="-5" pin="1"/>
@@
 <label x="55.88" y="190.5" size="1.27" layer="95" rot="R180" xref="yes"/>
 </segment>
+<segment>
+<pinref part="U2" gate="G$1" pin="INT"/>
+<wire x1="144.78" y1="190.5" x2="149.86" y2="190.5" width="0.1524" layer="91"/>
+<label x="149.86" y="190.5" size="1.778" layer="95" xref="yes"/>
+</segment>
 </net>
 <net name="XY-6" class="0">
@@
 <label x="55.88" y="187.96" size="1.27" layer="95" rot="R180" xref="yes"/>
 </segment>
+<segment>
+<wire x1="60.96" y1="170.18" x2="55.88" y2="170.18" width="0.1524" layer="91"/>
+<pinref part="J6" gate="-3" pin="1"/>
+<label x="55.88" y="170.18" size="1.27" layer="95" rot="R180" xref="yes"/>
+</segment>
 </net>
 <net name="XY-7" class="0">
@@
 <wire x1="60.96" y1="185.42" x2="55.88" y2="185.42" width="0.1524" layer="91"/>
 <label x="55.88" y="185.42" size="1.27" layer="95" rot="R180" xref="yes"/>
+</segment>
+<segment>
+<wire x1="60.96" y1="172.72" x2="55.88" y2="172.72" width="0.1524" layer="91"/>
+<pinref part="J6" gate="-2" pin="1"/>
+<label x="55.88" y="172.72" size="1.27" layer="95" rot="R180" xref="yes"/>
 </segment>
 </net>
@@
 <junction x="162.56" y="134.62"/>
 <label x="157.48" y="134.62" size="1.778" layer="95" rot="R180" xref="yes"/>
-<pinref part="C11" gate="G$1" pin="1"/>
+<pinref part="C9" gate="G$1" pin="1"/>
 <wire x1="170.18" y1="132.08" x2="170.18" y2="134.62" width="0.1524" layer="91"/>
 <pinref part="B1" gate="G$1" pin="+"/>

Commit message: Fix GPS module package so that all silkscreen markings are in top silkscreen layer Add a via in the SMA antenna ground pour. Move via in VBACK trace outside of battery holder outline to prevent possible short circuit. Revise date (10 December 2014) Correct battery voltage measurement calculation in schematic text.
Other:
- note added: "When VBAT=11.2V, voltage to ADC ~ VBAT/5 = 2.24V"
- note removed: "When VBAT=11.2V, voltage to ADC ~ VBAT/6 = 1.87V"
Changed lines of the file:
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@@
 (WAAS, EGNOS, GAGAN, MSAS) which requires no external input.</text>
 <text x="114.3" y="43.18" size="2.1844" layer="97">When VBAT=11.2V,
-voltage to ADC ~ VBAT/6 = 1.87V</text>
+voltage to ADC ~ VBAT/5 = 2.24V</text>
 <text x="73.66" y="12.7" size="2.1844" layer="97">MAX4173 has fixed output impedance of 12K
 100nF output cap C14 provides LPF, tau=1.2ms</text>

Commit message: Enlarge signal feed hole in center of SMA connector footprint. Available parts probably would not have fit if boards were run with previous footprint.
Parts:
- J4: device con-coax:BU-SMA-V -> pyIMU_GPS:BU-SMA-V
Changed lines of the file:
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@@
 <part name="GND9" library="supply1" deviceset="GND" device=""/>
 <part name="U3" library="pyIMU_GPS" deviceset="FGPMMOPA6H" device=""/>
-<part name="J4" library="con-coax" deviceset="BU-SMA-V" device=""/>
+<part name="J4" library="pyIMU_GPS" deviceset="BU-SMA-V" device=""/>
 <part name="GND4" library="supply1" deviceset="GND" device=""/>
 <part name="GND5" library="supply1" deviceset="GND" device=""/>
